Commit message: Fix Gazebo launch warnings and auto-load controllers
- Add dummy 'world' link to URDF to fix KDL root link inertia warning
- Remove redundant static_transform_publisher (now in URDF)
- Update launch file to auto-spawn controllers after entity spawn
- Use RegisterEventHandler for proper controller loading sequence
- Set controller update_rate to 1000Hz to match Gazebo physics rate
- Add allow_nonzero_velocity_at_trajectory_end: false to fix deprecation

Co-Authored-By: Claude Opus 4.5 <noreply@anthropic.com>

File: hpop_system/hpop_gazebo/urdf/chaser_satellite.urdf.xacro (robot description, xacro)
@@ -19,4 +19,11 @@
     <color rgba="0.8 0.2 0.2 1.0"/>
   </material>
+  <!-- Dummy root link (fixes KDL warning about inertia on root link) -->
+  <link name="world"/>
+  <joint name="world_to_base" type="fixed">
+    <parent link="world"/>
+    <child link="base_link"/>
+    <origin xyz="0 0 0" rpy="0 0 0"/>
+  </joint>
   <!-- Base link (satellite body) -->
   <link name="base_link">
