Commit message: Add satellite rendezvous simulation with HPOP integration (Phase 10)
- Add rendezvous_controller node for approach and docking control
- Implement Delta-V calculation and HPOP orbital mechanics integration
- Add Canadarm-style robot arm (2m reach, 6-DOF)
- Create satellite_mission.launch.py for integrated simulation
- Add MoveIt2 configuration (SRDF, kinematics, controllers)
- Add RViz configurations for docking and orbit views
- Add Mission Control Panel RViz plugin
- Update URDF: Canadarm arm for Chaser, remove solar panels from Target
- Add comprehensive README with architecture and sequence diagrams

Co-Authored-By: Claude Opus 4.5 <noreply@anthropic.com>

File: hpop_system/hpop_gazebo/urdf/chaser_satellite.urdf.xacro (robot description, xacro)
@@ -1,42 +1,46 @@
 <?xml version="1.0"?>
 <robot xmlns:xacro="http://www.ros.org/wiki/xacro" name="chaser_satellite">
-  <!-- Properties -->
-  <xacro:property name="satellite_mass" value="1000.0"/>
-  <xacro:property name="satellite_size_x" value="2.0"/>
-  <xacro:property name="satellite_size_y" value="1.5"/>
-  <xacro:property name="satellite_size_z" value="1.0"/>
+  <!-- Package path for config files -->
+  <xacro:property name="pkg_path" value="$(find hpop_gazebo)"/>
+  <!-- 6U CubeSat Properties (10cm x 20cm x 30cm - 2x3U config) -->
+  <xacro:property name="cubesat_unit" value="0.1"/>  <!-- 10cm = 1U -->
+  <xacro:property name="satellite_x" value="${cubesat_unit}"/>       <!-- 10cm -->
+  <xacro:property name="satellite_y" value="${2*cubesat_unit}"/>     <!-- 20cm (2U) -->
+  <xacro:property name="satellite_z" value="${3*cubesat_unit}"/>     <!-- 30cm (3U) -->
+  <xacro:property name="satellite_mass" value="12.0"/>  <!-- 12kg typical for 6U -->
+  <!-- Robot arm: Canadarm-style (thin and long, ~2m reach) -->
   <!-- Materials -->
-  <material name="gold">
-    <color rgba="0.9 0.8 0.2 1.0"/>
+  <material name="cubesat_body">
+    <color rgba="0.3 0.3 0.3 1.0"/>  <!-- Dark grey aluminum -->
+  </material>
+  <material name="solar_cell">
+    <color rgba="0.1 0.1 0.5 1.0"/>  <!-- Dark blue solar cells -->
   </material>
   <material name="grey">
-    <color rgba="0.5 0.5 0.5 1.0"/>
-  </material>
-  <material name="blue">
-    <color rgba="0.2 0.4 0.8 1.0"/>
+    <color rgba="0.6 0.6 0.6 1.0"/>
   </material>
   <material name="magnet_red">
-    <color rgba="0.8 0.2 0.2 1.0"/>
+    <color rgba="0.9 0.2 0.2 1.0"/>
   </material>
-  <!-- Dummy root link (fixes KDL warning about inertia on root link) -->
-  <link name="world"/>
-  <joint name="world_to_base" type="fixed">
-    <parent link="world"/>
+  <!-- Dummy root link for KDL (no inertia) -->
+  <link name="dummy_root"/>
+  <joint name="dummy_to_base" type="fixed">
+    <parent link="dummy_root"/>
     <child link="base_link"/>
     <origin xyz="0 0 0" rpy="0 0 0"/>
   </joint>
-  <!-- Base link (satellite body) -->
+  <!-- Base link (Large satellite body like ISS module) -->
   <link name="base_link">
     <visual>
       <origin xyz="0 0 0" rpy="0 0 0"/>
       <geometry>
-        <box size="${satellite_size_x} ${satellite_size_y} ${satellite_size_z}"/>
-      </geometry>
-      <material name="gold"/>
-    </visual>
-    <collision>
-      <origin xyz="0 0 0" rpy="0 0 0"/>
-      <geometry>
-        <box size="${satellite_size_x} ${satellite_size_y} ${satellite_size_z}"/>
+        <box size="${satellite_x} ${satellite_y} ${satellite_z}"/>
+      </geometry>
+      <material name="cubesat_body"/>
+    </visual>
+    <collision>
+      <origin xyz="0 0 0" rpy="0 0 0"/>
+      <geometry>
+        <box size="${satellite_x} ${satellite_y} ${satellite_z}"/>
       </geometry>
     </collision>
@@ -44,29 +48,29 @@
       <origin xyz="0 0 0" rpy="0 0 0"/>
       <mass value="${satellite_mass}"/>
-      <inertia ixx="${satellite_mass*(satellite_size_y*satellite_size_y+satellite_size_z*satellite_size_z)/12}"
+      <inertia ixx="${satellite_mass*(satellite_y*satellite_y+satellite_z*satellite_z)/12}"
                ixy="0" ixz="0"
-               iyy="${satellite_mass*(satellite_size_x*satellite_size_x+satellite_size_z*satellite_size_z)/12}"
+               iyy="${satellite_mass*(satellite_x*satellite_x+satellite_z*satellite_z)/12}"
                iyz="0"
-               izz="${satellite_mass*(satellite_size_x*satellite_size_x+satellite_size_y*satellite_size_y)/12}"/>
-    </inertial>
-  </link>
-  <!-- Solar panel 1 -->
+               izz="${satellite_mass*(satellite_x*satellite_x+satellite_y*satellite_y)/12}"/>
+    </inertial>
+  </link>
+  <!-- Deployable Solar Panel 1 (+Y side) - 6U size -->
   <link name="solar_panel_1">
     <visual>
       <origin xyz="0 0 0" rpy="0 0 0"/>
       <geometry>
-        <box size="3.0 0.05 1.5"/>
-      </geometry>
-      <material name="blue"/>
-    </visual>
-    <collision>
-      <origin xyz="0 0 0" rpy="0 0 0"/>
-      <geometry>
-        <box size="3.0 0.05 1.5"/>
-      </geometry>
-    </collision>
-    <inertial>
-      <mass value="50.0"/>
-      <inertia ixx="10" ixy="0" ixz="0" iyy="40" iyz="0" izz="40"/>
+        <box size="${satellite_z} 0.003 ${satellite_z*0.8}"/>
+      </geometry>
+      <material name="solar_cell"/>
+    </visual>
+    <collision>
+      <origin xyz="0 0 0" rpy="0 0 0"/>
+      <geometry>
+        <box size="${satellite_z} 0.003 ${satellite_z*0.8}"/>
+      </geometry>
+    </collision>
+    <inertial>
+      <mass value="0.3"/>
+      <inertia ixx="0.001" ixy="0" ixz="0" iyy="0.004" iyz="0" izz="0.004"/>
     </inertial>
   </link>
@@ -74,24 +78,24 @@
     <parent link="base_link"/>
     <child link="solar_panel_1"/>
-    <origin xyz="0 1.5 0" rpy="0 0 0"/>
-  </joint>
-  <!-- Solar panel 2 -->
+    <origin xyz="0 ${satellite_y/2 + satellite_z/2 + 0.005} 0" rpy="0 0 0"/>
+  </joint>
+  <!-- Deployable Solar Panel 2 (-Y side) - 6U size -->
   <link name="solar_panel_2">
     <visual>
       <origin xyz="0 0 0" rpy="0 0 0"/>
       <geometry>
-        <box size="3.0 0.05 1.5"/>
-      </geometry>
-      <material name="blue"/>
-    </visual>
-    <collision>
-      <origin xyz="0 0 0" rpy="0 0 0"/>
-      <geometry>
-        <box size="3.0 0.05 1.5"/>
-      </geometry>
-    </collision>
-    <inertial>
-      <mass value="50.0"/>
-      <inertia ixx="10" ixy="0" ixz="0" iyy="40" iyz="0" izz="40"/>
+        <box size="${satellite_z} 0.003 ${satellite_z*0.8}"/>
+      </geometry>
+      <material name="solar_cell"/>
+    </visual>
+    <collision>
+      <origin xyz="0 0 0" rpy="0 0 0"/>
+      <geometry>
+        <box size="${satellite_z} 0.003 ${satellite_z*0.8}"/>
+      </geometry>
+    </collision>
+    <inertial>
+      <mass value="0.3"/>
+      <inertia ixx="0.001" ixy="0" ixz="0" iyy="0.004" iyz="0" izz="0.004"/>
     </inertial>
   </link>
@@ -99,24 +103,24 @@
     <parent link="base_link"/>
     <child link="solar_panel_2"/>
-    <origin xyz="0 -1.5 0" rpy="0 0 0"/>
-  </joint>
-  <!-- Arm mounting point -->
+    <origin xyz="0 ${-satellite_y/2 - satellite_z/2 - 0.005} 0" rpy="0 0 0"/>
+  </joint>
+  <!-- Arm mounting point on +X face -->
   <link name="arm_base">
     <visual>
-      <origin xyz="0 0 0.05" rpy="0 0 0"/>
-      <geometry>
-        <cylinder radius="0.15" length="0.1"/>
-      </geometry>
-      <material name="grey"/>
-    </visual>
-    <collision>
-      <origin xyz="0 0 0.05" rpy="0 0 0"/>
-      <geometry>
-        <cylinder radius="0.15" length="0.1"/>
-      </geometry>
-    </collision>
-    <inertial>
-      <mass value="5.0"/>
-      <inertia ixx="0.1" ixy="0" ixz="0" iyy="0.1" iyz="0" izz="0.1"/>
+      <origin xyz="0 0 0.012" rpy="0 0 0"/>
+      <geometry>
+        <cylinder radius="0.02" length="0.024"/>
+      </geometry>
+      <material name="grey"/>
+    </visual>
+    <collision>
+      <origin xyz="0 0 0.012" rpy="0 0 0"/>
+      <geometry>
+        <cylinder radius="0.02" length="0.024"/>
+      </geometry>
+    </collision>
+    <inertial>
+      <mass value="0.1"/>
+      <inertia ixx="0.00002" ixy="0" ixz="0" iyy="0.00002" iyz="0" izz="0.00002"/>
     </inertial>
   </link>
@@ -124,28 +128,35 @@
     <parent link="base_link"/>
     <child link="arm_base"/>
-    <origin xyz="0.8 0 0.5" rpy="0 0 0"/>
+    <origin xyz="${satellite_x/2} 0 ${satellite_z/4}" rpy="0 ${pi/2} 0"/>
   </joint>
   <!-- =========================================== -->
-  <!-- OpenMANIPULATOR-P Robot Arm (6 DOF) -->
+  <!-- Canadarm-style Robot Arm (7 DOF) - Thin and Long -->
+  <!-- Total reach: ~2m (comparable to satellite scale) -->
   <!-- =========================================== -->
-  <!-- Link 1 -->
+  <!-- Arm dimensions (Canadarm-like proportions) -->
+  <xacro:property name="arm_tube_radius" value="0.015"/>  <!-- 15mm thin tube -->
+  <xacro:property name="joint_radius" value="0.025"/>     <!-- Joint housing -->
+  <xacro:property name="boom_length_1" value="0.6"/>      <!-- Upper boom: 60cm -->
+  <xacro:property name="boom_length_2" value="0.6"/>      <!-- Lower boom: 60cm -->
+  <xacro:property name="wrist_length" value="0.3"/>       <!-- Wrist section: 30cm -->
+  <!-- Link 1 (Base rotation housing) -->
   <link name="link1">
     <visual>
-      <origin xyz="0 0 0" rpy="0 0 0"/>
-      <geometry>
-        <mesh filename="package://hpop_gazebo/meshes/link1.stl" scale="0.001 0.001 0.001"/>
-      </geometry>
-      <material name="grey"/>
-    </visual>
-    <collision>
-      <origin xyz="0 0 0" rpy="0 0 0"/>
-      <geometry>
-        <mesh filename="package://hpop_gazebo/meshes/link1.stl" scale="0.001 0.001 0.001"/>
-      </geometry>
-    </collision>
-    <inertial>
-      <origin xyz="0.00023 0.00000 0.06223" rpy="0 0 0"/>
-      <mass value="0.85644"/>
-      <inertia ixx="0.00121" ixy="0.0" ixz="0.00001" iyy="0.00121" iyz="0.0" izz="0.00038"/>
+      <origin xyz="0 0 0.03" rpy="0 0 0"/>
+      <geometry>
+        <cylinder radius="${joint_radius}" length="0.06"/>
+      </geometry>
+      <material name="grey"/>
+    </visual>
+    <collision>
+      <origin xyz="0 0 0.03" rpy="0 0 0"/>
+      <geometry>
+        <cylinder radius="${joint_radius}" length="0.06"/>
+      </geometry>
+    </collision>
+    <inertial>
+      <origin xyz="0 0 0.03" rpy="0 0 0"/>
+      <mass value="0.3"/>
+      <inertia ixx="0.0001" ixy="0.0" ixz="0.0" iyy="0.0001" iyz="0.0" izz="0.00005"/>
     </inertial>
   </link>
@@ -153,219 +164,259 @@
     <parent link="arm_base"/>
     <child link="link1"/>
-    <origin xyz="0 0 0.1" rpy="0 0 0"/>
-  </joint>
-  <!-- Joint 1 -->
+    <origin xyz="0 0 0.024" rpy="0 0 0"/>
+  </joint>
+  <!-- Joint 1 (base yaw - rotation around Z) -->
   <joint name="joint1" type="revolute">
     <parent link="link1"/>
     <child link="link2"/>
-    <origin xyz="0.0 0.0 0.126" rpy="0 0 0"/>
+    <origin xyz="0.0 0.0 0.06" rpy="0 0 0"/>
     <axis xyz="0 0 1"/>
-    <limit velocity="6.5" effort="1000" lower="${-pi*0.9}" upper="${pi*0.9}"/>
-    <dynamics damping="0.7"/>
-  </joint>
-  <!-- Link 2 -->
+    <limit velocity="1.0" effort="50" lower="${-pi}" upper="${pi}"/>
+    <dynamics damping="1.0"/>
+  </joint>
+  <!-- Link 2 (Shoulder pitch joint housing) -->
   <link name="link2">
     <visual>
-      <origin xyz="0 0 0" rpy="0 0 0"/>
-      <geometry>
-        <mesh filename="package://hpop_gazebo/meshes/link2.stl" scale="0.001 0.001 0.001"/>
-      </geometry>
-      <material name="grey"/>
-    </visual>
-    <collision>
-      <origin xyz="0 0 0" rpy="0 0 0"/>
-      <geometry>
-        <mesh filename="package://hpop_gazebo/meshes/link2.stl" scale="0.001 0.001 0.001"/>
-      </geometry>
-    </collision>
-    <inertial>
-      <origin xyz="0.00000 0.00080 0.03183" rpy="0 0 0"/>
-      <mass value="0.94658"/>
-      <inertia ixx="0.00153" ixy="0.0" ixz="0.0" iyy="0.00046" iyz="-0.00001" izz="0.00152"/>
-    </inertial>
-  </link>
-  <!-- Joint 2 -->
+      <origin xyz="0 0 0.02" rpy="0 0 0"/>
+      <geometry>
+        <cylinder radius="${joint_radius}" length="0.04"/>
+      </geometry>
+      <material name="grey"/>
+    </visual>
+    <collision>
+      <origin xyz="0 0 0.02" rpy="0 0 0"/>
+      <geometry>
+        <cylinder radius="${joint_radius}" length="0.04"/>
+      </geometry>
+    </collision>
+    <inertial>
+      <origin xyz="0 0 0.02" rpy="0 0 0"/>
+      <mass value="0.2"/>
+      <inertia ixx="0.00005" ixy="0.0" ixz="0.0" iyy="0.00005" iyz="0.0" izz="0.00003"/>
+    </inertial>
+  </link>
+  <!-- Joint 2 (shoulder pitch) -->
   <joint name="joint2" type="revolute">
     <parent link="link2"/>
     <child link="link3"/>
-    <origin xyz="0.0 0.069 0.033" rpy="0 0 0"/>
+    <origin xyz="0.0 0.0 0.04" rpy="0 0 0"/>
     <axis xyz="0 1 0"/>
-    <limit velocity="6.5" effort="1000" lower="${-pi*0.5}" upper="${pi*0.5}"/>
-    <dynamics damping="0.7"/>
-  </joint>
-  <!-- Link 3 -->
+    <limit velocity="1.0" effort="50" lower="${-pi*0.75}" upper="${pi*0.75}"/>
+    <dynamics damping="1.0"/>
+  </joint>
+  <!-- Link 3 (Upper boom - long thin tube) -->
   <link name="link3">
     <visual>
-      <origin xyz="0 0 0" rpy="0 0 0"/>
-      <geometry>
-        <mesh filename="package://hpop_gazebo/meshes/link3.stl" scale="0.001 0.001 0.001"/>
-      </geometry>
-      <material name="grey"/>
-    </visual>
-    <collision>
-      <origin xyz="0 0 0" rpy="0 0 0"/>
-      <geometry>
-        <mesh filename="package://hpop_gazebo/meshes/link3.stl" scale="0.001 0.001 0.001"/>
-      </geometry>
-    </collision>
-    <inertial>
-      <origin xyz="0.01768 -0.06881 0.20524" rpy="0 0 0"/>
-      <mass value="1.30260"/>
-      <inertia ixx="0.01111" ixy="0.00001" ixz="-0.00134" iyy="0.01047" iyz="0.00016" izz="0.00202"/>
-    </inertial>
-  </link>
-  <!-- Joint 3 -->
+      <origin xyz="${boom_length_1/2} 0 0" rpy="0 ${pi/2} 0"/>
+      <geometry>
+        <cylinder radius="${arm_tube_radius}" length="${boom_length_1}"/>
+      </geometry>
+      <material name="grey"/>
+    </visual>
+    <collision>
+      <origin xyz="${boom_length_1/2} 0 0" rpy="0 ${pi/2} 0"/>
+      <geometry>
+        <cylinder radius="${arm_tube_radius}" length="${boom_length_1}"/>
+      </geometry>
+    </collision>
+    <inertial>
+      <origin xyz="${boom_length_1/2} 0 0" rpy="0 0 0"/>
+      <mass value="0.5"/>
+      <inertia ixx="0.0001" ixy="0.0" ixz="0.0" iyy="0.015" iyz="0.0" izz="0.015"/>
+    </inertial>
+  </link>
+  <!-- Joint 3 (elbow pitch) -->
   <joint name="joint3" type="revolute">
     <parent link="link3"/>
     <child link="link4"/>
-    <origin xyz="0.03000 -0.01150 0.26400" rpy="0 0 0"/>
+    <origin xyz="${boom_length_1} 0 0" rpy="0 0 0"/>
     <axis xyz="0 1 0"/>
-    <limit velocity="6.5" effort="1000" lower="${-pi*0.5}" upper="${pi*0.5}"/>
-    <dynamics damping="0.7"/>
-  </joint>
-  <!-- Link 4 -->
+    <limit velocity="1.0" effort="50" lower="${-pi*0.75}" upper="${pi*0.75}"/>
+    <dynamics damping="1.0"/>
+  </joint>
+  <!-- Link 4 (Elbow joint housing + Lower boom) -->
   <link name="link4">
-    <visual>
-      <origin xyz="0 0 0" rpy="0 0 0"/>
-      <geometry>
-        <mesh filename="package://hpop_gazebo/meshes/link4.stl" scale="0.001 0.001 0.001"/>
-      </geometry>
-      <material name="grey"/>
-    </visual>
-    <collision>
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
File: hpop_system/hpop_gazebo/urdf/target_satellite.urdf.xacro (robot description, xacro)
@@ -1,9 +1,10 @@
 <?xml version="1.0"?>
 <robot xmlns:xacro="http://www.ros.org/wiki/xacro" name="target_satellite">
-  <!-- Properties -->
-  <xacro:property name="satellite_mass" value="500.0"/>
-  <xacro:property name="satellite_size_x" value="1.5"/>
-  <xacro:property name="satellite_size_y" value="1.0"/>
-  <xacro:property name="satellite_size_z" value="1.0"/>
+  <!-- Properties - 3U CubeSat size (10cm x 10cm x 30cm) scaled for visualization -->
+  <xacro:property name="cubesat_unit" value="0.1"/>  <!-- 10cm = 1U -->
+  <xacro:property name="satellite_mass" value="5.0"/>  <!-- 5kg for 3U CubeSat -->
+  <xacro:property name="satellite_size_x" value="${cubesat_unit}"/>
+  <xacro:property name="satellite_size_y" value="${cubesat_unit}"/>
+  <xacro:property name="satellite_size_z" value="${3*cubesat_unit}"/>  <!-- 3U = 30cm -->
   <!-- Materials -->
   <material name="silver">
@@ -19,5 +20,15 @@
     <color rgba="0.2 0.8 0.2 1.0"/>
   </material>
-  <!-- Base link (satellite body) -->
+  <material name="target_orange">
+    <color rgba="1.0 0.5 0.0 1.0"/>
+  </material>
+  <!-- Dummy root link for KDL (no inertia) -->
+  <link name="target_dummy_root"/>
+  <joint name="target_dummy_to_base" type="fixed">
+    <parent link="target_dummy_root"/>
+    <child link="target_base_link"/>
+    <origin xyz="0 0 0" rpy="0 0 0"/>
+  </joint>
+  <!-- Base link (satellite body - 3U CubeSat) -->
   <link name="target_base_link">
     <visual>
@@ -44,63 +55,14 @@
     </inertial>
   </link>
-  <!-- Solar panel 1 -->
-  <link name="target_solar_panel_1">
-    <visual>
-      <origin xyz="0 0 0" rpy="0 0 0"/>
-      <geometry>
-        <box size="2.0 0.03 1.0"/>
-      </geometry>
-      <material name="solar_blue"/>
-    </visual>
-    <collision>
-      <origin xyz="0 0 0" rpy="0 0 0"/>
-      <geometry>
-        <box size="2.0 0.03 1.0"/>
-      </geometry>
-    </collision>
-    <inertial>
-      <mass value="30.0"/>
-      <inertia ixx="5" ixy="0" ixz="0" iyy="15" iyz="0" izz="15"/>
-    </inertial>
-  </link>
-  <joint name="target_solar_panel_1_joint" type="fixed">
-    <parent link="target_base_link"/>
-    <child link="target_solar_panel_1"/>
-    <origin xyz="0 1.0 0" rpy="0 0 0"/>
-  </joint>
-  <!-- Solar panel 2 -->
-  <link name="target_solar_panel_2">
-    <visual>
-      <origin xyz="0 0 0" rpy="0 0 0"/>
-      <geometry>
-        <box size="2.0 0.03 1.0"/>
-      </geometry>
-      <material name="solar_blue"/>
-    </visual>
-    <collision>
-      <origin xyz="0 0 0" rpy="0 0 0"/>
-      <geometry>
-        <box size="2.0 0.03 1.0"/>
-      </geometry>
-    </collision>
-    <inertial>
-      <mass value="30.0"/>
-      <inertia ixx="5" ixy="0" ixz="0" iyy="15" iyz="0" izz="15"/>
-    </inertial>
-  </link>
-  <joint name="target_solar_panel_2_joint" type="fixed">
-    <parent link="target_base_link"/>
-    <child link="target_solar_panel_2"/>
-    <origin xyz="0 -1.0 0" rpy="0 0 0"/>
-  </joint>
+  <!-- Solar panels removed - disabled debris satellite -->
   <!-- =========================================== -->
   <!-- Magnetic Docking Port (Target side) -->
   <!-- =========================================== -->
-  <!-- Docking port structure -->
+  <!-- Docking port structure (scaled for 3U CubeSat) -->
   <link name="docking_port">
     <visual>
       <origin xyz="0 0 0" rpy="0 0 0"/>
       <geometry>
-        <cylinder radius="0.1" length="0.15"/>
+        <cylinder radius="0.015" length="0.02"/>
       </geometry>
       <material name="dark_grey"/>
@@ -109,10 +71,10 @@
       <origin xyz="0 0 0" rpy="0 0 0"/>
       <geometry>
-        <cylinder radius="0.1" length="0.15"/>
+        <cylinder radius="0.015" length="0.02"/>
       </geometry>
     </collision>
     <inertial>
-      <mass value="5.0"/>
-      <inertia ixx="0.05" ixy="0" ixz="0" iyy="0.05" iyz="0" izz="0.05"/>
+      <mass value="0.1"/>
+      <inertia ixx="0.00001" ixy="0" ixz="0" iyy="0.00001" iyz="0" izz="0.00001"/>
     </inertial>
   </link>
@@ -120,5 +82,5 @@
     <parent link="target_base_link"/>
     <child link="docking_port"/>
-    <origin xyz="${satellite_size_x/2 + 0.075} 0 0" rpy="0 ${pi/2} 0"/>
+    <origin xyz="${satellite_size_x/2 + 0.01} 0 0" rpy="0 ${pi/2} 0"/>
   </joint>
   <!-- Magnetic contact surface -->
@@ -127,5 +89,5 @@
       <origin xyz="0 0 0" rpy="0 0 0"/>
       <geometry>
-        <cylinder radius="0.08" length="0.02"/>
+        <cylinder radius="0.012" length="0.005"/>
       </geometry>
       <material name="docking_green"/>
@@ -134,10 +96,10 @@
       <origin xyz="0 0 0" rpy="0 0 0"/>
       <geometry>
-        <cylinder radius="0.08" length="0.02"/>
+        <cylinder radius="0.012" length="0.005"/>
       </geometry>
     </collision>
     <inertial>
-      <mass value="0.5"/>
-      <inertia ixx="0.001" ixy="0" ixz="0" iyy="0.001" iyz="0" izz="0.001"/>
+      <mass value="0.02"/>
+      <inertia ixx="0.000001" ixy="0" ixz="0" iyy="0.000001" iyz="0" izz="0.000001"/>
     </inertial>
   </link>
@@ -145,37 +107,37 @@
     <parent link="docking_port"/>
     <child link="magnetic_contact_surface"/>
-    <origin xyz="0 0 0.085" rpy="0 0 0"/>
+    <origin xyz="0 0 0.012" rpy="0 0 0"/>
   </joint>
-  <!-- Antenna -->
-  <link name="antenna">
+  <!-- Antenna (scaled for 3U CubeSat) -->
+  <link name="target_antenna">
     <visual>
-      <origin xyz="0 0 0.15" rpy="0 0 0"/>
+      <origin xyz="0 0 0.03" rpy="0 0 0"/>
       <geometry>
-        <cylinder radius="0.02" length="0.3"/>
+        <cylinder radius="0.004" length="0.06"/>
       </geometry>
       <material name="dark_grey"/>
     </visual>
     <visual>
-      <origin xyz="0 0 0.35" rpy="0 0 0"/>
+      <origin xyz="0 0 0.07" rpy="0 0 0"/>
       <geometry>
-        <sphere radius="0.05"/>
+        <sphere radius="0.008"/>
       </geometry>
       <material name="silver"/>
     </visual>
     <collision>
-      <origin xyz="0 0 0.2" rpy="0 0 0"/>
+      <origin xyz="0 0 0.04" rpy="0 0 0"/>
       <geometry>
-        <cylinder radius="0.05" length="0.4"/>
+        <cylinder radius="0.01" length="0.08"/>
       </geometry>
     </collision>
     <inertial>
-      <mass value="2.0"/>
-      <inertia ixx="0.01" ixy="0" ixz="0" iyy="0.01" iyz="0" izz="0.01"/>
+      <mass value="0.02"/>
+      <inertia ixx="0.000001" ixy="0" ixz="0" iyy="0.000001" iyz="0" izz="0.000001"/>
     </inertial>
   </link>
-  <joint name="antenna_joint" type="fixed">
+  <joint name="target_antenna_joint" type="fixed">
     <parent link="target_base_link"/>
-    <child link="antenna"/>
-    <origin xyz="-0.3 0 ${satellite_size_z/2}" rpy="0 0 0"/>
+    <child link="target_antenna"/>
+    <origin xyz="-0.02 0 ${satellite_size_z/2}" rpy="0 0 0"/>
   </joint>
   <!-- =========================================== -->
@@ -183,12 +145,7 @@
   <!-- =========================================== -->
   <gazebo reference="target_base_link">
-    <material>Gazebo/Grey</material>
+    <material>Gazebo/Orange</material>
   </gazebo>
-  <gazebo reference="target_solar_panel_1">
-    <material>Gazebo/Blue</material>
-  </gazebo>
-  <gazebo reference="target_solar_panel_2">
-    <material>Gazebo/Blue</material>
-  </gazebo>
+  <!-- Solar panels removed -->
   <gazebo reference="docking_port">
     <material>Gazebo/DarkGrey</material>
@@ -197,3 +154,6 @@
     <material>Gazebo/Green</material>
   </gazebo>
+  <gazebo reference="target_antenna">
+    <material>Gazebo/Grey</material>
+  </gazebo>
 </robot>
